Commit message: added controller WIP

File: quadwheel/model/connector.xacro (robot description, xacro)
@@ -6,5 +6,5 @@
     <inertial>
       <origin xyz="0 0 -0.0286" rpy="0 0 0" />
-      <mass value="0.10"/>
+      <mass value="0.378"/>
       <inertia ixx="7.6e-5" ixy="0.0" ixz="0.0" iyy="7.6e-5" iyz="0.0" izz="0.000125"/>
     </inertial>

File: quadwheel/model/main.xacro (robot description, xacro)
@@ -7,4 +7,12 @@
     <parent link="base_link"/>
     <child link="chassis"/>
+    <origin xyz="0 0 0" rpy="0 0 0" />
+  </joint>
+  <!--Base Footprint-->
+  <link name="base_footprint" />
+  <joint name="base_to_footprint" type="fixed">
+    <parent link="base_link"/>
+    <child link="base_footprint"/>
+    <origin xyz="0 0 0" rpy="0 0 0" />
   </joint>
   <!-- Chassis -->
@@ -21,5 +29,5 @@
     <inertial>
       <origin xyz="0 0 0" rpy="0 0 0" />
-      <mass value="1"/>
+      <mass value="16.004"/>
       <inertia ixx="0.0001" ixy="0.0" ixz="0.0" iyy="0.0001" iyz="0.0" izz="0.0001"/>
     </inertial>

File: quadwheel/model/rim.xacro (robot description, xacro)
@@ -6,5 +6,5 @@
     <inertial>
       <origin xyz="0 0 -0.0182" rpy="0 0 0" />
-      <mass value="0.10"/>
+      <mass value="0.1"/>
       <inertia ixx="7.6e-5" ixy="0.0" ixz="0.0" iyy="7.6e-5" iyz="0.0" izz="0.000125"/>
     </inertial>

File: quadwheel/model/roller.xacro (robot description, xacro)
@@ -6,5 +6,5 @@
       <origin xyz="0 0 0" rpy="0 0 0" />
       <inertia ixx="1e-6" ixy="0.0" ixz="0.0" iyy="1e-6" iyz="0.0" izz="1e-7"/>
-      <mass value="0.010"/>
+      <mass value="0.001"/>
     </inertial>
     <visual>

File: quadwheel/model/ros2_control.xacro (robot description, xacro)
@@ -40,5 +40,5 @@
     <gazebo>
         <plugin name="gz_ros2_control::GazeboSimROS2ControlPlugin" filename="gz_ros2_control-system">
-            <parameters>$(find quadwheel)/config/my_controllers.yaml</parameters>
+            <parameters>$(find quadwheel)/config/omni_controller.yaml</parameters>
         </plugin>
     </gazebo>

Commit message: wheel updates

File: quadwheel/model/connector.xacro (robot description, xacro)
@@ -6,6 +6,6 @@
     <inertial>
       <origin xyz="0 0 -0.0286" rpy="0 0 0" />
-      <mass value="0.378"/>
-      <inertia ixx="7.6e-5" ixy="0.0" ixz="0.0" iyy="7.6e-5" iyz="0.0" izz="0.000125"/>
+      <mass value="0.092"/>
+      <inertia ixx="4.8343e-05" ixy="0.0" ixz="0.0" iyy="4.8343e-05" iyz="0.0" izz="4.6517e-05"/>
     </inertial>
     <visual>

File: quadwheel/model/main.xacro (robot description, xacro)
@@ -1,52 +1,10 @@
 <?xml version='1.0'?>
 <robot name="4_wheel_omni" xmlns:xacro="http://www.ros.org/wiki/xacro">
-  <xacro:include filename="$(find quadwheel)/model/connector.xacro"/>
-  <!-- World Link -->
-  <link name="base_link" />
-  <joint name="base_to_chassis" type="fixed">
-    <parent link="base_link"/>
-    <child link="chassis"/>
-    <origin xyz="0 0 0" rpy="0 0 0" />
-  </joint>
-  <!--Base Footprint-->
-  <link name="base_footprint" />
-  <joint name="base_to_footprint" type="fixed">
-    <parent link="base_link"/>
-    <child link="base_footprint"/>
-    <origin xyz="0 0 0" rpy="0 0 0" />
-  </joint>
-  <!-- Chassis -->
-  <link name="chassis">
-    <visual>
-      <origin xyz="0 0 0" rpy="0 0 0" />
-      <geometry>
-        <mesh filename="file://$(find quadwheel)/meshes/chassis.stl" />
-      </geometry>
-      <material name="">
-        <color rgba="1 1 0 1" />
-      </material>
-    </visual>
-    <inertial>
-      <origin xyz="0 0 0" rpy="0 0 0" />
-      <mass value="16.004"/>
-      <inertia ixx="0.0001" ixy="0.0" ixz="0.0" iyy="0.0001" iyz="0.0" izz="0.0001"/>
-    </inertial>
-  </link>
-  <gazebo reference="chassis">
-    <visual>
-      <material>
-        <ambient>0.9 0.9 0 1</ambient>
-        <diffuse>0.9 0.9 0 1</diffuse>
-        <specular>0.9 0.9 0 1</specular>
-      </material>
-    </visual>
-  </gazebo>
-  <!--Wheel Rims -->
-  <xacro:connector name="1" parent="chassis" xyz="0.228 0.228 0.01" rpy="1.57 0 -0.7854"/>
-  <xacro:connector name="2" parent="chassis" xyz="0.228 -0.228 0.01" rpy="1.57 0 -2.3562"/>
-  <xacro:connector name="3" parent="chassis" xyz="-0.228 -0.228 0.01" rpy="1.57 0 -3.9270"/>
-  <xacro:connector name="4" parent="chassis" xyz="-0.228 0.228 0.01" rpy="1.57 0 -5.4978"/>
+  <!-- Robot -->
+  <xacro:include filename="$(find quadwheel)/model/chassis.xacro"/>
   <!-- Control -->
   <xacro:include filename="$(find quadwheel)/model/ros2_control.xacro"/>
-  <!--Include The Arm-->
+  <!-- Cameras -->
+  <!--<xacro:include filename="$(find quadwheel)/model/cameras.xacro"/>-->
+  <!-- Arm -->
 </robot>

File: quadwheel/model/rim.xacro (robot description, xacro)
@@ -6,11 +6,11 @@
     <inertial>
       <origin xyz="0 0 -0.0182" rpy="0 0 0" />
-      <mass value="0.1"/>
-      <inertia ixx="7.6e-5" ixy="0.0" ixz="0.0" iyy="7.6e-5" iyz="0.0" izz="0.000125"/>
+      <mass value="0.20"/>
+      <inertia ixx="6.3068e-04" ixy="0.0" ixz="0.0" iyy="6.3068e-04" iyz="0.0" izz="0.0012"/>
     </inertial>
     <visual>
       <origin xyz="0 0 -0.0182" rpy="0 0 0" />
       <geometry>
-        <cylinder radius="0.050" length="0.0364"/>
+        <cylinder radius="0.076" length="0.0381"/>
       </geometry>
     </visual>
@@ -22,22 +22,24 @@
     <origin xyz = "${xyz}" rpy = "${rpy}"/>
   </joint>
-<xacro:roller name="1" parent="${name}"  xyz="0.0415 0 -0.0284" rpy="1.57 0 0"/>
-<xacro:roller name="2" parent="${name}"  xyz="0.0390 0.0142 -0.008" rpy="1.57 0 0.3491"/>
-<xacro:roller name="3" parent="${name}"  xyz="0.0318 0.0267 -0.0284" rpy="1.57 0 0.6981"/>
-<xacro:roller name="4" parent="${name}"  xyz="0.0208 0.0359 -0.008" rpy="1.57 0 1.0472"/>
-<xacro:roller name="5" parent="${name}"  xyz="0.0072 0.0409 -0.0284" rpy="1.57 0 1.3963"/>
-<xacro:roller name="6" parent="${name}"  xyz="-0.0072 0.0409 -0.008" rpy="1.57 0 1.7453"/>
-<xacro:roller name="7" parent="${name}"  xyz="-0.0208 0.0359 -0.0284" rpy="1.57 0 2.0944"/>
-<xacro:roller name="8" parent="${name}"  xyz="-0.0318 0.0267 -0.008" rpy="1.57 0 2.4435"/>
-<xacro:roller name="9" parent="${name}"  xyz="-0.0390 0.0142 -0.0284" rpy="1.57 0 2.7925"/>
-<xacro:roller name="10" parent="${name}"  xyz="-0.0415 0 -0.008" rpy="1.57 0 3.1416"/>
-<xacro:roller name="11" parent="${name}"  xyz="-0.0390 -0.0142 -0.0284" rpy="1.57 0 3.4907"/>
-<xacro:roller name="12" parent="${name}"  xyz="-0.0318 -0.0267 -0.008" rpy="1.57 0 3.8397"/>
-<xacro:roller name="13" parent="${name}"  xyz="-0.0208 -0.0359 -0.0284" rpy="1.57 0 4.1888"/>
-<xacro:roller name="14" parent="${name}"  xyz="-0.00072 -0.0409 -0.008" rpy="1.57 0 4.5379"/>
-<xacro:roller name="15" parent="${name}"  xyz="0.0072 -0.0409 -0.0284" rpy="1.57 0 4.8869"/>
-<xacro:roller name="16" parent="${name}"  xyz="0.0208 -0.0359 -0.008" rpy="1.57 0 5.2360"/>
-<xacro:roller name="17" parent="${name}"  xyz="0.0318 -0.0267 -0.0284" rpy="1.57 0 5.5851"/>
-<xacro:roller name="18" parent="${name}"  xyz="0.0390 -0.0142 -0.008" rpy="1.57 0 5.9341"/>
+<xacro:roller name="1" parent="${name}"  xyz="0.068 0 -0.0091" rpy="1.57 0 0"/>
+<xacro:roller name="2" parent="${name}"  xyz="0.0647 0.021 -0.0291" rpy="1.57 0 0.3142"/>
+<xacro:roller name="3" parent="${name}"  xyz="0.055 0.04 -0.0091" rpy="1.57 0 0.6283"/>
+<xacro:roller name="4" parent="${name}"  xyz="0.04 0.055 -0.0291" rpy="1.57 0 0.9425"/>
+<xacro:roller name="5" parent="${name}"  xyz="0.021 0.0647 -0.0091" rpy="1.57 0 1.2566"/>
+<xacro:roller name="6" parent="${name}"  xyz="0 0.068 -0.0291" rpy="1.57 0 1.5708"/>
+<xacro:roller name="7" parent="${name}"  xyz="-0.021 0.0647 -0.0091" rpy="1.57 0 1.8850"/>
+<xacro:roller name="8" parent="${name}"  xyz="-0.04 0.055 -0.0291" rpy="1.57 0 2.1991"/>
+<xacro:roller name="9" parent="${name}"  xyz="-0.055 0.04 -0.0091" rpy="1.57 0 2.5133"/>
+<xacro:roller name="10" parent="${name}"  xyz="-0.0647 0.021 -0.0291" rpy="1.57 0 2.8274"/>
+<xacro:roller name="11" parent="${name}"  xyz="-0.068 0 -0.0091" rpy="1.57 0 3.1416"/>
+<xacro:roller name="12" parent="${name}"  xyz="-0.0647 -0.021 -0.0291" rpy="1.57 0 3.4558"/>
+<xacro:roller name="13" parent="${name}"  xyz="-0.055 -0.04 -0.0091" rpy="1.57 0 3.7699"/>
+<xacro:roller name="14" parent="${name}"  xyz="-0.04 -0.055 -0.0291" rpy="1.57 0 4.0841"/>
+<xacro:roller name="15" parent="${name}"  xyz="-0.021 -0.0647 -0.0091" rpy="1.57 0 4.3982"/>
+<xacro:roller name="16" parent="${name}"  xyz="0 -0.068 -0.0291" rpy="1.57 0 4.7124"/>
+<xacro:roller name="17" parent="${name}"  xyz="0.021 -0.0647 -0.0091" rpy="1.57 0 5.0265"/>
+<xacro:roller name="18" parent="${name}"  xyz="0.04 -0.055 -0.0291" rpy="1.57 0 5.3407"/>
+<xacro:roller name="19" parent="${name}"  xyz="0.055 -0.04 -0.0091" rpy="1.57 0 5.6549"/>
+<xacro:roller name="20" parent="${name}"  xyz="0.0647 -0.021 -0.0291" rpy="1.57 0 5.9690"/>
 <gazebo reference="rim_${name}_link">
   <visual>

File: quadwheel/model/roller.xacro (robot description, xacro)
@@ -5,6 +5,6 @@
     <inertial>
       <origin xyz="0 0 0" rpy="0 0 0" />
-      <inertia ixx="1e-6" ixy="0.0" ixz="0.0" iyy="1e-6" iyz="0.0" izz="1e-7"/>
-      <mass value="0.001"/>
+      <inertia ixx="1e-6" ixy="0.0" ixz="0.0" iyy="1e-6" iyz="0.0" izz="1e-6"/>
+      <mass value="0.01"/>
     </inertial>
     <visual>
