Commit message: Gazebo and Rviz Mismatch FIX

File: quadwheel/model/chassis.xacro (robot description, xacro)
@@ -12,6 +12,6 @@
   <link name="base_footprint" />
   <joint name="base_to_footprint" type="fixed">
-    <parent link="base_link"/>
-    <child link="base_footprint"/>
+    <parent link="base_footprint"/>
+    <child link="base_link"/>
     <origin xyz="0 0 0" rpy="0 0 0" />
   </joint>
@@ -43,7 +43,7 @@
   </gazebo>
   <!--Wheel Rims -->
-  <xacro:connector name="1" parent="chassis" xyz="0.228 0.228 0.01" rpy="1.57 0 -0.7854"/>
-  <xacro:connector name="2" parent="chassis" xyz="0.228 -0.228 0.01" rpy="1.57 0 -2.3562"/>
-  <xacro:connector name="3" parent="chassis" xyz="-0.228 -0.228 0.01" rpy="1.57 0 -3.9270"/>
-  <xacro:connector name="4" parent="chassis" xyz="-0.228 0.228 0.01" rpy="1.57 0 -5.4978"/>
+  <xacro:connector name="1" parent="chassis" xyz="0.228 0.228 0.01" rpy="1.57 0 2.3562"/>  <!--Front Left-->
+  <xacro:connector name="2" parent="chassis" xyz="0.228 -0.228 0.01" rpy="1.57 0 0.7838"/> <!--Front Right-->
+  <xacro:connector name="3" parent="chassis" xyz="-0.228 -0.228 0.01" rpy="1.57 0 -0.7838"/>  <!--Back Right-->
+  <xacro:connector name="4" parent="chassis" xyz="-0.228 0.228 0.01" rpy="1.57 0 -2.3562"/> <!--Back Left -->
 </robot>

File: quadwheel/model/connector.xacro (robot description, xacro)
@@ -5,10 +5,10 @@
   <link name="C${name}">
     <inertial>
-      <origin xyz="0 0 -0.0286" rpy="0 0 0" />
+      <origin xyz="0 0 0.0286" rpy="0 0 0" />
       <mass value="0.092"/>
       <inertia ixx="4.8343e-05" ixy="0.0" ixz="0.0" iyy="4.8343e-05" iyz="0.0" izz="4.6517e-05"/>
     </inertial>
     <visual>
-      <origin xyz="0 0 -0.0286" rpy="0 0 0" />
+      <origin xyz="0 0 0.0286" rpy="0 0 0" />
       <geometry>
         <cylinder radius="0.0318" length="0.0572"/>
@@ -23,5 +23,5 @@
   </joint>
   <!-- Wheel Rims -->
-  <xacro:rim name="wheel_${name}" parent="C${name}" xyz="0 0 -0.0572" rpy="0 0 0"/>
+  <xacro:rim name="wheel_${name}" parent="C${name}" xyz="0 0 0.0572" rpy="0 0 0"/>
   <gazebo reference="C${name}">
     <visual>

File: quadwheel/model/rim.xacro (robot description, xacro)
@@ -5,10 +5,10 @@
   <link name="rim_${name}_link">
     <inertial>
-      <origin xyz="0 0 -0.0182" rpy="0 0 0" />
+      <origin xyz="0 0 0.0182" rpy="0 0 0" />
       <mass value="0.20"/>
       <inertia ixx="6.3068e-04" ixy="0.0" ixz="0.0" iyy="6.3068e-04" iyz="0.0" izz="0.0012"/>
     </inertial>
     <visual>
-      <origin xyz="0 0 -0.0182" rpy="0 0 0" />
+      <origin xyz="0 0 0.0182" rpy="0 0 0" />
       <geometry>
         <cylinder radius="0.076" length="0.0381"/>
@@ -22,24 +22,24 @@
     <origin xyz = "${xyz}" rpy = "${rpy}"/>
   </joint>
-<xacro:roller name="1" parent="${name}"  xyz="0.068 0 -0.0091" rpy="1.57 0 0"/>
-<xacro:roller name="2" parent="${name}"  xyz="0.0647 0.021 -0.0291" rpy="1.57 0 0.3142"/>
-<xacro:roller name="3" parent="${name}"  xyz="0.055 0.04 -0.0091" rpy="1.57 0 0.6283"/>
-<xacro:roller name="4" parent="${name}"  xyz="0.04 0.055 -0.0291" rpy="1.57 0 0.9425"/>
-<xacro:roller name="5" parent="${name}"  xyz="0.021 0.0647 -0.0091" rpy="1.57 0 1.2566"/>
-<xacro:roller name="6" parent="${name}"  xyz="0 0.068 -0.0291" rpy="1.57 0 1.5708"/>
-<xacro:roller name="7" parent="${name}"  xyz="-0.021 0.0647 -0.0091" rpy="1.57 0 1.8850"/>
-<xacro:roller name="8" parent="${name}"  xyz="-0.04 0.055 -0.0291" rpy="1.57 0 2.1991"/>
-<xacro:roller name="9" parent="${name}"  xyz="-0.055 0.04 -0.0091" rpy="1.57 0 2.5133"/>
-<xacro:roller name="10" parent="${name}"  xyz="-0.0647 0.021 -0.0291" rpy="1.57 0 2.8274"/>
-<xacro:roller name="11" parent="${name}"  xyz="-0.068 0 -0.0091" rpy="1.57 0 3.1416"/>
-<xacro:roller name="12" parent="${name}"  xyz="-0.0647 -0.021 -0.0291" rpy="1.57 0 3.4558"/>
-<xacro:roller name="13" parent="${name}"  xyz="-0.055 -0.04 -0.0091" rpy="1.57 0 3.7699"/>
-<xacro:roller name="14" parent="${name}"  xyz="-0.04 -0.055 -0.0291" rpy="1.57 0 4.0841"/>
-<xacro:roller name="15" parent="${name}"  xyz="-0.021 -0.0647 -0.0091" rpy="1.57 0 4.3982"/>
-<xacro:roller name="16" parent="${name}"  xyz="0 -0.068 -0.0291" rpy="1.57 0 4.7124"/>
-<xacro:roller name="17" parent="${name}"  xyz="0.021 -0.0647 -0.0091" rpy="1.57 0 5.0265"/>
-<xacro:roller name="18" parent="${name}"  xyz="0.04 -0.055 -0.0291" rpy="1.57 0 5.3407"/>
-<xacro:roller name="19" parent="${name}"  xyz="0.055 -0.04 -0.0091" rpy="1.57 0 5.6549"/>
-<xacro:roller name="20" parent="${name}"  xyz="0.0647 -0.021 -0.0291" rpy="1.57 0 5.9690"/>
+<xacro:roller name="1" parent="${name}"  xyz="0.068 0 0.0091" rpy="1.57 0 0"/>
+<xacro:roller name="2" parent="${name}"  xyz="0.0647 0.021 0.0291" rpy="1.57 0 0.3142"/>
+<xacro:roller name="3" parent="${name}"  xyz="0.055 0.04 0.0091" rpy="1.57 0 0.6283"/>
+<xacro:roller name="4" parent="${name}"  xyz="0.04 0.055 0.0291" rpy="1.57 0 0.9425"/>
+<xacro:roller name="5" parent="${name}"  xyz="0.021 0.0647 0.0091" rpy="1.57 0 1.2566"/>
+<xacro:roller name="6" parent="${name}"  xyz="0 0.068 0.0291" rpy="1.57 0 1.5708"/>
+<xacro:roller name="7" parent="${name}"  xyz="-0.021 0.0647 0.0091" rpy="1.57 0 1.8850"/>
+<xacro:roller name="8" parent="${name}"  xyz="-0.04 0.055 0.0291" rpy="1.57 0 2.1991"/>
+<xacro:roller name="9" parent="${name}"  xyz="-0.055 0.04 0.0091" rpy="1.57 0 2.5133"/>
+<xacro:roller name="10" parent="${name}"  xyz="-0.0647 0.021 0.0291" rpy="1.57 0 2.8274"/>
+<xacro:roller name="11" parent="${name}"  xyz="-0.068 0 0.0091" rpy="1.57 0 3.1416"/>
+<xacro:roller name="12" parent="${name}"  xyz="-0.0647 -0.021 0.0291" rpy="1.57 0 3.4558"/>
+<xacro:roller name="13" parent="${name}"  xyz="-0.055 -0.04 0.0091" rpy="1.57 0 3.7699"/>
+<xacro:roller name="14" parent="${name}"  xyz="-0.04 -0.055 0.0291" rpy="1.57 0 4.0841"/>
+<xacro:roller name="15" parent="${name}"  xyz="-0.021 -0.0647 0.0091" rpy="1.57 0 4.3982"/>
+<xacro:roller name="16" parent="${name}"  xyz="0 -0.068 0.0291" rpy="1.57 0 4.7124"/>
+<xacro:roller name="17" parent="${name}"  xyz="0.021 -0.0647 0.0091" rpy="1.57 0 5.0265"/>
+<xacro:roller name="18" parent="${name}"  xyz="0.04 -0.055 0.0291" rpy="1.57 0 5.3407"/>
+<xacro:roller name="19" parent="${name}"  xyz="0.055 -0.04 0.0091" rpy="1.57 0 5.6549"/>
+<xacro:roller name="20" parent="${name}"  xyz="0.0647 -0.021 0.0291" rpy="1.57 0 5.9690"/>
 <gazebo reference="rim_${name}_link">
   <visual>
