Commit message: Dockerfile and reformat

File: roam_base/model/chassis.xacro (robot description, xacro)
@@ -1,5 +1,5 @@
 <?xml version='1.0'?>
 <robot xmlns:xacro="http://www.ros.org/wiki/xacro">
-  <xacro:include filename="$(find quadwheel)/model/connector.xacro"/>
+  <xacro:include filename="$(find roam_base)/model/connector.xacro"/>
   <!-- World Link -->
   <link name="base_link" />
@@ -21,5 +21,5 @@
       <origin xyz="0 0 0" rpy="0 0 0" />
       <geometry>
-        <mesh filename="file://$(find quadwheel)/meshes/chassis.stl" />
+        <mesh filename="file://$(find roam_base)/meshes/chassis.stl" />
       </geometry>
       <material name="">

File: roam_base/model/connector.xacro (robot description, xacro)
@@ -1,5 +1,5 @@
 <?xml version='1.0'?>
 <robot xmlns:xacro="http://www.ros.org/wiki/xacro">
-<xacro:include filename="$(find quadwheel)/model/rim.xacro"/>
+<xacro:include filename="$(find roam_base)/model/rim.xacro"/>
 <xacro:macro name="connector" params="name parent xyz rpy">
   <link name="C${name}">

File: roam_base/model/rim.xacro (robot description, xacro)
@@ -1,5 +1,5 @@
 <?xml version='1.0'?>
 <robot xmlns:xacro="http://www.ros.org/wiki/xacro">
-<xacro:include filename="$(find quadwheel)/model/roller.xacro"/>
+<xacro:include filename="$(find roam_base)/model/roller.xacro"/>
 <xacro:macro name="rim" params="name parent xyz rpy">
   <link name="rim_${name}_link">

File: roam_base/model/ros2_control.xacro (robot description, xacro)
@@ -40,5 +40,5 @@
     <gazebo>
         <plugin name="gz_ros2_control::GazeboSimROS2ControlPlugin" filename="gz_ros2_control-system">
-            <parameters>$(find quadwheel)/config/omni_controller.yaml</parameters>
+            <parameters>$(find roam_base)/config/omni_controller.yaml</parameters>
         </plugin>
     </gazebo>
