Commit message: motors with format

File: roam_arduino_hardware/model/main.xacro (robot description, xacro)
@@ -2,5 +2,5 @@
 <robot name="roam_base" xmlns:xacro="http://www.ros.org/wiki/xacro">
   <!-- Robot -->
-  <xacro:include filename="$(find roam_base)/model/chassis.xacro"/>
+  <xacro:include filename="$(find roam_base_description)/model/chassis.xacro"/>
   <!-- Control -->
   <xacro:include filename="$(find roam_arduino_hardware)/model/ros2_control.xacro"/>

File: roam_base_description/model/chassis.xacro (robot description, xacro)
@@ -1,5 +1,5 @@
 <?xml version='1.0'?>
 <robot xmlns:xacro="http://www.ros.org/wiki/xacro">
-  <xacro:include filename="$(find roam_base)/model/connector.xacro"/>
+  <xacro:include filename="$(find roam_base_description)/model/connector.xacro"/>
   <!-- World Link -->
   <link name="base_link" />
@@ -21,5 +21,5 @@
       <origin xyz="0 0 0" rpy="0 0 0" />
       <geometry>
-        <mesh filename="file://$(find roam_base)/meshes/chassis.stl" />
+        <mesh filename="file://$(find roam_base_description)/meshes/chassis.stl" />
       </geometry>
       <material name="">

File: roam_base_description/model/connector.xacro (robot description, xacro)
@@ -1,5 +1,5 @@
 <?xml version='1.0'?>
 <robot xmlns:xacro="http://www.ros.org/wiki/xacro">
-<xacro:include filename="$(find roam_base)/model/rim.xacro"/>
+<xacro:include filename="$(find roam_base_description)/model/rim.xacro"/>
 <xacro:macro name="connector" params="name parent xyz rpy">
   <link name="C${name}">

File: roam_base_description/model/rim.xacro (robot description, xacro)
@@ -1,5 +1,5 @@
 <?xml version='1.0'?>
 <robot xmlns:xacro="http://www.ros.org/wiki/xacro">
-<xacro:include filename="$(find roam_base)/model/roller.xacro"/>
+<xacro:include filename="$(find roam_base_description)/model/roller.xacro"/>
 <xacro:macro name="rim" params="name parent xyz rpy">
   <link name="rim_${name}_link">

File: roam_base_gazebo/model/ros2_control.xacro (robot description, xacro)
@@ -40,5 +40,5 @@
     <gazebo>
         <plugin name="gz_ros2_control::GazeboSimROS2ControlPlugin" filename="gz_ros2_control-system">
-            <parameters>$(find roam_base)/config/omni_controller.yaml</parameters>
+            <parameters>$(find roam_base_gazebo)/config/omni_controller.yaml</parameters>
         </plugin>
     </gazebo>
