Commit message: reformat/moveit inprogress

File: roam/roam_base_description/model/chassis.xacro (robot description, xacro)
@@ -2,18 +2,4 @@
 <robot xmlns:xacro="http://www.ros.org/wiki/xacro">
   <xacro:include filename="$(find roam_base_description)/model/connector.xacro"/>
-  <!-- World Link -->
-  <link name="base_link" />
-  <joint name="base_to_chassis" type="fixed">
-    <parent link="base_link"/>
-    <child link="chassis"/>
-    <origin xyz="0 0 0" rpy="0 0 0" />
-  </joint>
-  <!--Base Footprint-->
-  <link name="base_footprint" />
-  <joint name="base_to_footprint" type="fixed">
-    <parent link="base_footprint"/>
-    <child link="base_link"/>
-    <origin xyz="0 0 0" rpy="0 0 0" />
-  </joint>
   <!-- Chassis -->
   <link name="chassis">
