Commit message: moveit(arm+base) + gazebo

File: roam/roam_base_description/model/main.xacro (robot description, xacro)
@@ -11,10 +11,9 @@
   </joint>
   <!-- Base Footprint -->
-  <link name="base_footprint" />
-  <joint name="base_to_footprint" type="fixed">
+  <!--<joint name="base_to_footprint" type="fixed">
     <parent link="base_footprint"/>
     <child link="base_link"/>
     <origin xyz="0 0 0" rpy="0 0 0" />
-  </joint>
+  </joint> -->
   <!-- Cameras -->
   <!--<xacro:include filename="$(find quadwheel)/model/cameras.xacro"/>-->

File: roam/roam_base_gazebo/model/main.xacro (robot description, xacro)
@@ -12,18 +12,11 @@
   </joint>
   <!--Base Footprint-->
-  <link name="base_footprint" />
+  <!--<link name="base_footprint" />
   <joint name="base_to_footprint" type="fixed">
     <parent link="base_footprint"/>
     <child link="base_link"/>
     <origin xyz="0 0 0" rpy="0 0 0" />
-  </joint>
+  </joint> -->
   <!-- Cameras -->
   <!--<xacro:include filename="$(find quadwheel)/model/cameras.xacro"/>-->
-  <!-- Arm -->
-  <!--<xacro:include filename="$(find annin_ar4_description)/urdf/ar_gazebo.urdf.xacro"/>-->
-  <!--<joint name="arm_mount_joint" type="fixed">
-    <parent link="chassis_link"/>
-    <child link="ar4_base_link"/>
-    <origin xyz="0 0 0.4" rpy="0 0 0" />
-  </joint> -->
 </robot>

File: roam_moveit/model/roam_urdf.ros2_control.xacro (robot description, xacro)
@@ -7,4 +7,17 @@
               <plugin>gz_ros2_control/GazeboSimSystem</plugin>
             </hardware>
+            <!-- Fake Control Joints -->
+            <joint name="base_x">
+              <command_interface name="position"/>
+              <state_interface name="position"/>
+            </joint>
+            <joint name="base_y">
+              <command_interface name="position"/>
+              <state_interface name="position"/>
+            </joint>
+            <joint name="base_theta">
+              <command_interface name="position"/>
+              <state_interface name="position"/>
+            </joint>
             <!-- Base -->
             <joint name="chassis_C1_joint">

File: roam_moveit/model/roam_urdf.urdf.xacro (robot description, xacro)
@@ -4,4 +4,49 @@
     <!-- Import roam_urdf urdf file -->
     <xacro:include filename="$(find roam_base_description)/model/main.xacro" />
+    <!-- X linear joint -->
+    <link name="base_footprint" >
+        <inertial>
+        <mass value="0.001"/>
+        <origin xyz="0 0 0"/>
+        <inertia ixx="0.00001" iyy="0.00001" izz="0.00001" ixy="0" ixz="0" iyz="0"/>
+        </inertial>
+    </link>
+    <link name="base_x_link">
+        <inertial>
+        <mass value="0.001"/>
+        <origin xyz="0 0 0"/>
+        <inertia ixx="0.00001" iyy="0.00001" izz="0.00001" ixy="0" ixz="0" iyz="0"/>
+        </inertial>
+    </link>
+    <joint name="base_x" type="prismatic">
+        <parent link="base_footprint"/>
+        <child link="base_x_link"/>
+        <origin xyz="0 0 0" rpy="0 0 0"/>
+        <axis xyz="1 0 0"/>
+        <limit effort="0.01" velocity="1.5" lower="-10.0" upper="10.0"/>
+    </joint>
+    <!-- Y linear joint -->
+    <link name="base_y_link">
+        <inertial>
+        <mass value="0.001"/>
+        <origin xyz="0 0 0"/>
+        <inertia ixx="0.00001" iyy="0.00001" izz="0.00001" ixy="0" ixz="0" iyz="0"/>
+        </inertial>
+    </link>
+    <joint name="base_y" type="prismatic">
+        <parent link="base_x_link"/>
+        <child link="base_y_link"/>
+        <origin xyz="0 0 0" rpy="0 0 0"/>
+        <axis xyz="0 1 0"/>
+        <limit effort="0.01" velocity="1.5" lower="-10.0" upper="10.0"/>
+    </joint>
+    <!-- Theta rotational joint -->
+    <joint name="base_theta" type="continuous">
+        <parent link="base_y_link"/>
+        <child link="base_link"/>
+        <origin xyz="0 0 0" rpy="0 0 0"/>
+        <axis xyz="0 0 1"/>
+        <limit effort="0.01" velocity="6.0"/>
+    </joint>
     <!-- Import control_xacro -->
     <xacro:include filename="roam_urdf.ros2_control.xacro" />
