Commit message: moveit + gazebo

File: roam_moveit/model/roam_urdf.ros2_control.xacro (robot description, xacro)
@@ -5,7 +5,40 @@
         <ros2_control name="${name}" type="system">
             <hardware>
-                <!-- By default, set up controllers for simulation. This won't work on real hardware -->
-                <plugin>mock_components/GenericSystem</plugin>
+              <plugin>gz_ros2_control/GazeboSimSystem</plugin>
             </hardware>
+            <!-- Base -->
+            <joint name="chassis_C1_joint">
+              <command_interface name="velocity">
+                <param name="min">-100</param>
+                <param name="max">100</param>
+              </command_interface>
+              <state_interface name="velocity"/>
+              <state_interface name="position"/>
+            </joint>
+            <joint name="chassis_C2_joint">
+              <command_interface name="velocity">
+                <param name="min">-100</param>
+                <param name="max">100</param>
+              </command_interface>
+              <state_interface name="velocity"/>
+              <state_interface name="position"/>
+            </joint>
+            <joint name="chassis_C3_joint">
+              <command_interface name="velocity">
+                <param name="min">-100</param>
+                <param name="max">100</param>
+              </command_interface>
+              <state_interface name="velocity"/>
+              <state_interface name="position"/>
+              </joint>
+            <joint name="chassis_C4_joint">
+              <command_interface name="velocity">
+                <param name="min">-100</param>
+                <param name="max">100</param>
+              </command_interface>
+              <state_interface name="velocity"/>
+              <state_interface name="position"/>
+            </joint>
+            <!-- Arm -->
             <joint name="arm_joint_1">
                 <command_interface name="position"/>
@@ -57,4 +90,9 @@
             </joint>
         </ros2_control>
+        <gazebo>
+          <plugin name="gz_ros2_control::GazeboSimROS2ControlPlugin" filename="libgz_ros2_control-system.so">
+            <parameters>$(find roam_moveit)/config/ros2_controllers.yaml</parameters>
+          </plugin>
+        </gazebo>
     </xacro:macro>
 </robot>

File: roam_moveit/model/roam_urdf.urdf.xacro (robot description, xacro)
@@ -6,4 +6,4 @@
     <!-- Import control_xacro -->
     <xacro:include filename="roam_urdf.ros2_control.xacro" />
-    <xacro:roam_urdf_ros2_control name="FakeSystem" initial_positions_file="$(arg initial_positions_file)"/>
+    <xacro:roam_urdf_ros2_control name="GazeboSystem" initial_positions_file="$(arg initial_positions_file)"/>
 </robot>
