Commit message: moveit + gazebo (no sliding now)

File: roam_moveit/model/roam_urdf.urdf.xacro (robot description, xacro)
@@ -4,19 +4,27 @@
     <!-- Import roam_urdf urdf file -->
     <xacro:include filename="$(find roam_base_description)/model/main.xacro" />
-    <!-- X linear joint -->
-    <link name="base_footprint" >
-        <inertial>
+    <!-- Base virtual links -->
+    <link name="base_footprint">
+    <inertial>
         <mass value="0.001"/>
-        <origin xyz="0 0 0"/>
+        <origin xyz="0 0 0" rpy="0 0 0"/>
         <inertia ixx="0.00001" iyy="0.00001" izz="0.00001" ixy="0" ixz="0" iyz="0"/>
-        </inertial>
+    </inertial>
     </link>
     <link name="base_x_link">
-        <inertial>
+    <inertial>
         <mass value="0.001"/>
-        <origin xyz="0 0 0"/>
+        <origin xyz="0 0 0" rpy="0 0 0"/>
         <inertia ixx="0.00001" iyy="0.00001" izz="0.00001" ixy="0" ixz="0" iyz="0"/>
-        </inertial>
+    </inertial>
     </link>
+    <link name="base_y_link">
+    <inertial>
+        <mass value="0.001"/>
+        <origin xyz="0 0 0" rpy="0 0 0"/>
+        <inertia ixx="0.00001" iyy="0.00001" izz="0.00001" ixy="0" ixz="0" iyz="0"/>
+    </inertial>
+    </link>
+    <!-- X linear joint -->
     <joint name="base_x" type="prismatic">
         <parent link="base_footprint"/>
@@ -24,14 +32,8 @@
         <origin xyz="0 0 0" rpy="0 0 0"/>
         <axis xyz="1 0 0"/>
-        <limit effort="0.01" velocity="1.5" lower="-10.0" upper="10.0"/>
+        <!-- Fake limits for MoveIt -->
+        <limit effort="1e-6" velocity="1e-6" lower="-10" upper="10"/>
     </joint>
     <!-- Y linear joint -->
-    <link name="base_y_link">
-        <inertial>
-        <mass value="0.001"/>
-        <origin xyz="0 0 0"/>
-        <inertia ixx="0.00001" iyy="0.00001" izz="0.00001" ixy="0" ixz="0" iyz="0"/>
-        </inertial>
-    </link>
     <joint name="base_y" type="prismatic">
         <parent link="base_x_link"/>
@@ -39,5 +41,5 @@
         <origin xyz="0 0 0" rpy="0 0 0"/>
         <axis xyz="0 1 0"/>
-        <limit effort="0.01" velocity="1.5" lower="-10.0" upper="10.0"/>
+        <limit effort="1e-6" velocity="1e-6" lower="-10" upper="10"/>
     </joint>
     <!-- Theta rotational joint -->
@@ -47,5 +49,4 @@
         <origin xyz="0 0 0" rpy="0 0 0"/>
         <axis xyz="0 0 1"/>
-        <limit effort="0.01" velocity="6.0"/>
     </joint>
     <!-- Import control_xacro -->
