Commit message: moves with path

File: rome_description/rome_base_description/model/chassis.xacro (robot description, xacro)
@@ -16,5 +16,5 @@
       <origin xyz="0 0 0" rpy="0 0 0" />
       <mass value="16.004"/>
-      <inertia ixx="0.0001" ixy="0.0" ixz="0.0" iyy="0.0001" iyz="0.0" izz="0.0001"/>
+      <inertia ixx="0.3610" ixy="0.0" ixz="0.0" iyy="0.3610" iyz="0.0" izz="0.6749"/>
     </inertial>
   </link>

File: rome_description/rome_base_description/model/main.xacro (robot description, xacro)
@@ -15,5 +15,5 @@
     <parent link="chassis"/>
     <child link="arm_base_link"/>
-    <origin xyz="0 0 0." rpy="0 0 0" />
+    <origin xyz="0 0 0.133" rpy="0 0 0" />
   </joint>
 </robot>
