Commit message: predefense-push

File: ar4/annin_ar4_description/urdf/ar_macro.xacro (robot description, xacro)
@@ -168,5 +168,5 @@
         upper="${robot_parameters['j4_limit_max']}"
         effort="-1"
-        velocity="1.0472"
+        velocity="0"
       />
     </joint>

File: rome_description/rome_arm_description/model/arm_urdf.xacro (robot description, xacro)
@@ -153,6 +153,6 @@
       <axis xyz="0 0 -1"/>
       <limit
-        lower="-180"
-        upper="180"
+        lower="0"
+        upper="0"
         effort="-1"
         velocity="1.0472"

File: rome_moveit/model/rome_gazebo.ros2_control.xacro (robot description, xacro)
@@ -1,5 +1,5 @@
 <?xml version="1.0"?>
 <robot xmlns:xacro="http://www.ros.org/wiki/xacro">
-    <xacro:macro name="rome_urdf_ros2_control" params="name initial_positions_file">
+    <xacro:macro name="rome_urdf_ros2_control_gz" params="name initial_positions_file">
         <xacro:property name="initial_positions" value="${xacro.load_yaml(initial_positions_file)['initial_positions']}"/>
         <ros2_control name="${name}" type="system">

File: rome_moveit/model/rome_physical.ros2_control.xacro (robot description, xacro)
@@ -1,6 +1,7 @@
 <?xml version="1.0"?>
 <robot xmlns:xacro="http://www.ros.org/wiki/xacro">
-    <xacro:macro name="rome_urdf_ros2_control" params="name initial_positions_file">
+    <xacro:macro name="rome_urdf_ros2_control_real" params="name initial_positions_file joint_offset_parameters_file base_port arm_port">
         <xacro:property name="initial_positions" value="${xacro.load_yaml(initial_positions_file)['initial_positions']}"/>
+        <xacro:property name="joint_offset_parameters" value="${xacro.load_yaml(joint_offset_parameters_file)}"/>
         <ros2_control name="${name}_fake_base" type="system">
             <hardware>
@@ -22,4 +23,8 @@
         </ros2_control>
         <ros2_control name="${name}_base" type="system">
+          <hardware>
+            <plugin>rome_arduino_hardware/ROMEARD</plugin>
+            <param name="port">/dev/ttyACM2</param>
+          </hardware>
             <!-- Base -->
             <joint name="chassis_C1_joint">
@@ -55,4 +60,15 @@
               <state_interface name="position"/>
             </joint>
+        </ros2_control>
+        <ros2_control name="${name}_arm" type="system">
+          <hardware>
+            <plugin>mock_components/GenericSystem</plugin>
+            <!--<plugin>annin_ar4_driver/ARHardwareInterface</plugin>
+            <param name="serial_port">/dev/ttyACM0</param>
+            <param name="ar_model">mk3</param>
+            <param name="calibrate">False</param>
+            <param name="calib_sequence">0012345</param>
+            <param name="velocity_control_enabled">False</param>-->
+          </hardware>
             <!-- Arm -->
             <joint name="arm_joint_1">
@@ -63,4 +79,5 @@
                 </state_interface>
                 <state_interface name="velocity"/>
+                <param name="position_offset">${joint_offset_parameters['joint_1']}</param>
             </joint>
             <joint name="arm_joint_2">
@@ -71,4 +88,5 @@
                 </state_interface>
                 <state_interface name="velocity"/>
+                <param name="position_offset">${joint_offset_parameters['joint_2']}</param>
             </joint>
             <joint name="arm_joint_3">
@@ -79,4 +97,5 @@
                 </state_interface>
                 <state_interface name="velocity"/>
+                <param name="position_offset">${joint_offset_parameters['joint_3']}</param>
             </joint>
             <joint name="arm_joint_4">
@@ -87,4 +106,5 @@
                 </state_interface>
                 <state_interface name="velocity"/>
+                <param name="position_offset">${joint_offset_parameters['joint_4']}</param>
             </joint>
             <joint name="arm_joint_5">
@@ -95,4 +115,5 @@
                 </state_interface>
                 <state_interface name="velocity"/>
+                <param name="position_offset">${joint_offset_parameters['joint_5']}</param>
             </joint>
             <joint name="arm_joint_6">
@@ -103,4 +124,5 @@
                 </state_interface>
                 <state_interface name="velocity"/>
+                <param name="position_offset">${joint_offset_parameters['joint_6']}</param>
             </joint>
         </ros2_control>

File: rome_moveit/model/rome_urdf.urdf.xacro (robot description, xacro)
@@ -3,4 +3,6 @@
     <xacro:arg name="initial_positions_file" default="initial_positions.yaml" />
     <xacro:arg name="hardware" default="gazebo"/>
+    <xacro:arg name="base_port" default="0"/>
+    <xacro:arg name="arm_port" default="0"/>
     <xacro:property name="hardware" value="$(arg hardware)" />
     <!-- Import rome_urdf urdf file -->
@@ -55,9 +57,14 @@
     <xacro:if value="${hardware == 'gazebo'}">
         <xacro:include filename="rome_gazebo.ros2_control.xacro" />
-        <xacro:rome_urdf_ros2_control name="GazeboSystem" initial_positions_file="$(arg initial_positions_file)"/>
+        <xacro:rome_urdf_ros2_control_gz name="GazeboSystem" initial_positions_file="$(arg initial_positions_file)"/>
     </xacro:if>
     <xacro:if value="${hardware == 'real'}">
         <xacro:include filename="rome_physical.ros2_control.xacro" />
-        <xacro:rome_urdf_ros2_control name="RealSystem" initial_positions_file="$(arg initial_positions_file)"/>
+        <xacro:rome_urdf_ros2_control_real name="RealSystem"
+            initial_positions_file="$(arg initial_positions_file)"
+            base_port="$(arg base_port)"
+            arm_port="$(arg arm_port)"
+            joint_offset_parameters_file="$(find annin_ar4_driver)/config/joint_offsets/mk3.yaml"
+        />
     </xacro:if>
 </robot>
